Commit message: 🏷️ Rename to Simple Drone

File: urdf/x3.urdf (robot description, URDF)
Before this commit: robot x3, 6 links, 5 joints
Links:
- link base_link: geometry collision box size=0.47 0.47 0.11; visual mesh filename=package://simple_drone_description/meshes/x3.dae scale=1 1 1
- link rotor_0: geometry collision cylinder length=0.005 radius=0.1; visual mesh filename=package://simple_drone_description/meshes/propeller_ccw.dae scale=0.1 0.1 0.1
- link rotor_1: geometry collision cylinder length=0.005 radius=0.1; visual mesh filename=package://simple_drone_description/meshes/propeller_ccw.dae scale=0.1 0.1 0.1
- link rotor_2: geometry collision cylinder length=0.005 radius=0.1; visual mesh filename=package://simple_drone_description/meshes/propeller_cw.dae scale=0.1 0.1 0.1
- link rotor_3: geometry collision cylinder length=0.005 radius=0.1; visual mesh filename=package://simple_drone_description/meshes/propeller_cw.dae scale=0.1 0.1 0.1
